File: eagle/Nixies/Numishnik/numishnik.brd (EAGLE design)
At the start: 65.1 x 37.5 mm, 43 parts, among them IC1 MBI5026GP, IC2 MBI5026GP, IC6 DS3234, IC7 MEGA8-AI, SW1 BUTTON-IT_1181, X1 USB-MICROB, X3 53047-06

Commit message: added xtal, changed rtcsel#.. not routed
Parts:
- added TP3, TP4: TPSPAD1-13, 0-svo:P1-13
Connections:
- new net N$1: IC7.7, TP3.1
- new net XTAL2: IC7.8, TP4.1
- net RTCSEL#: now also IC7.11; no longer IC7.7
Changed lines of the file:
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@@
 <grid distance="2.5" unitdist="mil" unit="mm" style="dots" multiple="1" display="yes" altdistance="0.1" altunitdist="mm" altunit="mm"/>
 <layers>
-<layer number="1" name="Top" color="4" fill="1" visible="no" active="yes"/>
+<layer number="1" name="Top" color="4" fill="1" visible="yes" active="yes"/>
 <layer number="16" name="Bottom" color="1" fill="1" visible="yes" active="yes"/>
 <layer number="17" name="Pads" color="2" fill="1" visible="yes" active="yes"/>
@@
 <layer number="19" name="Unrouted" color="6" fill="1" visible="no" active="yes"/>
 <layer number="20" name="Dimension" color="15" fill="1" visible="yes" active="yes"/>
-<layer number="21" name="tPlace" color="7" fill="1" visible="no" active="yes"/>
-<layer number="22" name="bPlace" color="7" fill="1" visible="no" active="yes"/>
-<layer number="23" name="tOrigins" color="15" fill="1" visible="no" active="yes"/>
-<layer number="24" name="bOrigins" color="15" fill="1" visible="no" active="yes"/>
+<layer number="21" name="tPlace" color="7" fill="1" visible="yes" active="yes"/>
+<layer number="22" name="bPlace" color="7" fill="1" visible="yes" active="yes"/>
+<layer number="23" name="tOrigins" color="15" fill="1" visible="yes" active="yes"/>
+<layer number="24" name="bOrigins" color="15" fill="1" visible="yes" active="yes"/>
 <layer number="25" name="tNames" color="7" fill="1" visible="no" active="yes"/>
-<layer number="26" name="bNames" color="7" fill="1" visible="no" active="yes"/>
+<layer number="26" name="bNames" color="7" fill="1" visible="yes" active="yes"/>
 <layer number="27" name="tValues" color="7" fill="1" visible="no" active="yes"/>
-<layer number="28" name="bValues" color="7" fill="1" visible="no" active="yes"/>
+<layer number="28" name="bValues" color="7" fill="1" visible="yes" active="yes"/>
 <layer number="29" name="tStop" color="7" fill="3" visible="no" active="yes"/>
 <layer number="30" name="bStop" color="7" fill="6" visible="no" active="yes"/>
@@
 <layer number="50" name="dxf" color="7" fill="1" visible="no" active="no"/>
 <layer number="51" name="tDocu" color="7" fill="1" visible="no" active="yes"/>
-<layer number="52" name="bDocu" color="7" fill="1" visible="no" active="yes"/>
+<layer number="52" name="bDocu" color="7" fill="1" visible="yes" active="yes"/>
 <layer number="53" name="tGND_GNDA" color="7" fill="9" visible="no" active="no"/>
 <layer number="54" name="bGND_GNDA" color="1" fill="9" visible="no" active="no"/>
@@
 <element name="R12" library="rcl" package="R0805-SVO" value="000" x="35.56" y="17.78" rot="MR315"/>
 <element name="R13" library="rcl" package="R0805-SVO" value="000" x="30.7975" y="15.71625" rot="MR225"/>
+<element name="TP3" library="0-svo" package="P1-13" value="TPSPAD1-13" x="-4.1275" y="-3.81"/>
+<element name="TP4" library="0-svo" package="P1-13" value="TPSPAD1-13" x="-4.1275" y="-7.8105"/>
 </elements>
 <signals>
@@
 </signal>
 <signal name="RTCSEL#">
-<contactref element="IC7" pad="7"/>
 <contactref element="IC6" pad="1"/>
-<wire x1="29.8404625" y1="7.903884375" x2="29.811384375" y2="7.903884375" width="0.254" layer="16"/>
 <wire x1="13.97" y1="3.81" x2="13.97" y2="3.02" width="0.254" layer="16"/>
 <wire x1="29.811384375" y1="7.903884375" x2="29.05125" y2="7.14375" width="0.3048" layer="16"/>
@@
 <wire x1="21.9075" y1="3.65125" x2="14.12875" y2="3.65125" width="0.254" layer="16"/>
 <wire x1="14.12875" y1="3.65125" x2="13.97" y2="3.81" width="0.254" layer="16"/>
+<contactref element="IC7" pad="11"/>
+<wire x1="29.811384375" y1="7.903884375" x2="30.406146875" y2="11.711796875" width="0" layer="19" extent="16-16"/>
 </signal>
 <signal name="BTNSET">
@@
 <wire x1="32.0675" y1="25.0825" x2="27.94" y2="29.21" width="0.3048" layer="16"/>
 </signal>
+<signal name="XTAL2">
+<contactref element="IC7" pad="8"/>
+<contactref element="TP4" pad="1"/>
+<wire x1="-4.1275" y1="-7.8105" x2="29.274775" y2="8.469571875" width="0" layer="19" extent="16-16"/>
+</signal>
+<signal name="N$1">
+<contactref element="IC7" pad="7"/>
+<contactref element="TP3" pad="1"/>
+<wire x1="-4.1275" y1="-3.81" x2="29.8404625" y2="7.903884375" width="0" layer="19" extent="16-16"/>
+</signal>
 </signals>

Commit message: latest version, not all fixes fully fixed: careful with SS
Connections:
- removed net BTN+: IC7.28
- removed net BTNSET: IC7.27
- net +5V: no longer IC7.20
Routing:
- net +5V: track 145.8 -> 144.3 mm
Changed lines of the file:
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@@
 <contactref element="C11" pad="1"/>
 <contactref element="IC7" pad="18"/>
-<contactref element="IC7" pad="20"/>
 <contactref element="IC7" pad="4"/>
 <contactref element="IC7" pad="6"/>
@@
 <wire x1="34.76625" y1="12.85875" x2="35.8775" y2="11.7475" width="0.3048" layer="16"/>
 <wire x1="35.8775" y1="11.7475" x2="35.946815625" y2="11.7475" width="0.254" layer="16"/>
-<wire x1="35.946815625" y1="11.7475" x2="37.042484375" y2="12.84316875" width="0.3048" layer="16"/>
 <wire x1="37.481284375" y1="14.588715625" x2="36.52529375" y2="14.588715625" width="0.3048" layer="16"/>
 <wire x1="36.52529375" y1="14.588715625" x2="35.911115625" y2="13.9745375" width="0.3048" layer="16"/>
@@
 <wire x1="29.811384375" y1="7.903884375" x2="30.406146875" y2="11.711796875" width="0" layer="19" extent="16-16"/>
 </signal>
-<signal name="BTNSET">
-<contactref element="IC7" pad="27"/>
-</signal>
-<signal name="BTN+">
-<contactref element="IC7" pad="28"/>
-</signal>
 <signal name="N$4">
