File: projects/zloshnik/eagle/Zloshnik/zloshnikrev1.sch (EAGLE design)
At the start: 56 parts, among them IC2 78L05F, IC7 MEGA8-AI, Q1 IRLML2502, Q2 IRLML2502, Q3 IRLML2502, SW1 BUTTON-IT_1181

Commit message: read_dsn.py only pads no rotation
Parts:
- removed Q3: IRLML2502, xmaker:IRLML2502
- removed TP1, TP2, TP3, TP4, TP5, TP6: (no value), wirepad:1,6/0,8
- added C8, C9: 0,01 1kV, 0-rcl:C-EUC2220K
- added D5, D6: (no value), semicon-smd-ipc:D-SOD-87
- added Q4: IRF630N, transistor-power:IRF740
- added R10, R8, R9: 33K, rcl:R-EU_R0805S
- C12: value 1.0 -> 0,01 2kV; device rcl:C-EUC0805S -> 0-rcl:C-EUC1812
- C7: value 0,01 1kV -> 0,01 2kV
- Q2: value IRLML2502 -> IRF630N; device xmaker:IRLML2502 -> transistor-power:IRF740
- R2: value 470K -> 33K
- R3: value 4K7 -> 33K
- R6: value 100k -> 33K; device 0-rcl:R-EU_0207/7 -> rcl:R-EU_R0805S
Connections:
- removed net +1KV: C7.2, R6.2
- removed net HV+: R2.1
- removed net N$8: TP3.P, TP4.P
- new net +300V: C7.2, R9.1
- new net -600V: C12.2, R10.1
- new net N$11: R6.1, R8.2
- new net N$14: C8.1, D5.A, D6.C
- new net N$17: C19.2, C9.1, D12.A, D5.C
- new net N$18: R10.2, R3.1
- net +5V: no longer D3.C
- net FBACK: no longer C12.1, D3.AC, R2.2, R3.2
- net GND: now also C12.1, C19.1, D11.C, Q4.S; no longer C12.2, D3.A, Q3.S, R3.1
- net N$1: now also Q2.G; no longer Q3.G
- net N$12: now also R2.1, R3.2; no longer C18.2, D11.C, D12.A
- net N$13: now also R6.2; no longer C19.1, D11.A
- net N$15: now also C9.2, D6.A, R2.2; no longer C19.2, D12.C, R6.1
- net N$16: now also C18.2
- net N$2: now also Q4.D; no longer Q2.D
- net N$3: now also Q4.G; no longer Q2.G
- net N$4: now also Q2.D; no longer Q3.D
- net N$6: no longer C18.1
- net N$7: now also C18.1, C8.2, D11.A, D12.C; no longer TP1.P, TP2.P
- net N$9: now also R8.1, R9.2; no longer TP5.P, TP6.P
Other:
- moved on the sheet: C12, C16, C17, C18, C19, C7, D10, D11, D12, D9, R2, R3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
