File: projects/zloshnik/eagle/Zloshnik/zloshnik2.sch (EAGLE design)
At the start: 111 parts, among them IC1 TL5626D, IC2 78L05F, IC3 REG1117, IC6 DS3234, IC7 MEGA8-AI, Q2 IRF630N, Q4 IRF630N, SW1 BUTTON-IT_1181

Commit message: just updated los values on the schematic
Parts:
- removed R39: (no value), 0-rcl:R-TRIMM3314J
- removed R47: (no value), 0-rcl:R-TRIMMTS63Z
- R22, R30: value 2M2 -> 33K
Other:
- note added: "todo: add jumper here"
Changed lines of the file:
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@@
 <grid distance="0.1" unitdist="inch" unit="inch" style="lines" multiple="1" display="no" altdistance="0.01" altunitdist="inch" altunit="inch"/>
 <layers>
-<layer number="1" name="Top" color="4" fill="1" visible="yes" active="no"/>
-<layer number="16" name="Bottom" color="1" fill="1" visible="yes" active="no"/>
-<layer number="17" name="Pads" color="2" fill="1" visible="yes" active="no"/>
-<layer number="18" name="Vias" color="2" fill="1" visible="yes" active="no"/>
-<layer number="19" name="Unrouted" color="6" fill="1" visible="yes" active="no"/>
-<layer number="20" name="Dimension" color="15" fill="1" visible="yes" active="no"/>
-<layer number="21" name="tPlace" color="7" fill="1" visible="yes" active="no"/>
-<layer number="22" name="bPlace" color="7" fill="1" visible="yes" active="no"/>
-<layer number="23" name="tOrigins" color="15" fill="1" visible="yes" active="no"/>
-<layer number="24" name="bOrigins" color="15" fill="1" visible="yes" active="no"/>
-<layer number="25" name="tNames" color="7" fill="1" visible="yes" active="no"/>
-<layer number="26" name="bNames" color="7" fill="1" visible="yes" active="no"/>
-<layer number="27" name="tValues" color="7" fill="1" visible="yes" active="no"/>
-<layer number="28" name="bValues" color="7" fill="1" visible="yes" active="no"/>
+<layer number="1" name="Top" color="4" fill="1" visible="no" active="no"/>
+<layer number="16" name="Bottom" color="1" fill="1" visible="no" active="no"/>
+<layer number="17" name="Pads" color="2" fill="1" visible="no" active="no"/>
+<layer number="18" name="Vias" color="2" fill="1" visible="no" active="no"/>
+<layer number="19" name="Unrouted" color="6" fill="1" visible="no" active="no"/>
+<layer number="20" name="Dimension" color="15" fill="1" visible="no" active="no"/>
+<layer number="21" name="tPlace" color="7" fill="1" visible="no" active="no"/>
+<layer number="22" name="bPlace" color="7" fill="1" visible="no" active="no"/>
+<layer number="23" name="tOrigins" color="15" fill="1" visible="no" active="no"/>
+<layer number="24" name="bOrigins" color="15" fill="1" visible="no" active="no"/>
+<layer number="25" name="tNames" color="7" fill="1" visible="no" active="no"/>
+<layer number="26" name="bNames" color="7" fill="1" visible="no" active="no"/>
+<layer number="27" name="tValues" color="7" fill="1" visible="no" active="no"/>
+<layer number="28" name="bValues" color="7" fill="1" visible="no" active="no"/>
 <layer number="29" name="tStop" color="7" fill="3" visible="no" active="no"/>
 <layer number="30" name="bStop" color="7" fill="6" visible="no" active="no"/>
@@
 <layer number="35" name="tGlue" color="7" fill="4" visible="no" active="no"/>
 <layer number="36" name="bGlue" color="7" fill="5" visible="no" active="no"/>
-<layer number="37" name="tTest" color="7" fill="1" visible="yes" active="no"/>
-<layer number="38" name="bTest" color="7" fill="1" visible="yes" active="no"/>
+<layer number="37" name="tTest" color="7" fill="1" visible="no" active="no"/>
+<layer number="38" name="bTest" color="7" fill="1" visible="no" active="no"/>
 <layer number="39" name="tKeepout" color="4" fill="11" visible="no" active="no"/>
 <layer number="40" name="bKeepout" color="1" fill="11" visible="no" active="no"/>
@@
 <layer number="44" name="Drills" color="7" fill="1" visible="no" active="no"/>
 <layer number="45" name="Holes" color="7" fill="1" visible="no" active="no"/>
-<layer number="46" name="Milling" color="3" fill="1" visible="yes" active="no"/>
-<layer number="47" name="Measures" color="7" fill="1" visible="yes" active="no"/>
-<layer number="48" name="Document" color="7" fill="1" visible="yes" active="no"/>
-<layer number="49" name="Reference" color="7" fill="1" visible="yes" active="no"/>
-<layer number="50" name="dxf" color="7" fill="1" visible="yes" active="no"/>
-<layer number="51" name="tDocu" color="7" fill="1" visible="yes" active="no"/>
-<layer number="52" name="bDocu" color="7" fill="1" visible="yes" active="no"/>
-<layer number="53" name="tGND_GNDA" color="7" fill="9" visible="yes" active="no"/>
-<layer number="54" name="bGND_GNDA" color="1" fill="9" visible="yes" active="no"/>
-<layer number="56" name="wert" color="7" fill="1" visible="yes" active="no"/>
+<layer number="46" name="Milling" color="3" fill="1" visible="no" active="no"/>
+<layer number="47" name="Measures" color="7" fill="1" visible="no" active="no"/>
+<layer number="48" name="Document" color="7" fill="1" visible="no" active="no"/>
+<layer number="49" name="Reference" color="7" fill="1" visible="no" active="no"/>
+<layer number="50" name="dxf" color="7" fill="1" visible="no" active="no"/>
+<layer number="51" name="tDocu" color="7" fill="1" visible="no" active="no"/>
+<layer number="52" name="bDocu" color="7" fill="1" visible="no" active="no"/>
+<layer number="53" name="tGND_GNDA" color="7" fill="9" visible="no" active="no"/>
+<layer number="54" name="bGND_GNDA" color="1" fill="9" visible="no" active="no"/>
+<layer number="56" name="wert" color="7" fill="1" visible="no" active="no"/>
 <layer number="91" name="Nets" color="2" fill="1" visible="yes" active="yes"/>
 <layer number="92" name="Busses" color="1" fill="1" visible="yes" active="yes"/>
@@
 <part name="R20" library="0-rcl" deviceset="R-TRIMM" device="4G/J" value="10K"/>
 <part name="R21" library="0-rcl" deviceset="R-TRIMM" device="4G/J" value="500K"/>
-<part name="R22" library="rcl" deviceset="R-EU_" device="R0805S" value="2M2"/>
+<part name="R22" library="rcl" deviceset="R-EU_" device="R0805S" value="33K"/>
 <part name="R23" library="rcl" deviceset="R-EU_" device="R0805S" value="0"/>
 <part name="GND19" library="supply1" deviceset="GND" device=""/>
@@
 <part name="R28" library="0-rcl" deviceset="R-TRIMM" device="4G/J" value="10K"/>
 <part name="R29" library="0-rcl" deviceset="R-TRIMM" device="4G/J" value="500K"/>
-<part name="R30" library="rcl" deviceset="R-EU_" device="R0805S" value="2M2"/>
+<part name="R30" library="rcl" deviceset="R-EU_" device="R0805S" value="33K"/>
 <part name="R31" library="rcl" deviceset="R-EU_" device="R0805S" value="0"/>
 <part name="GND24" library="supply1" deviceset="GND" device=""/>
@@
 <part name="CAP-" library="wirepad" deviceset="2,54/0,8" device=""/>
 <part name="CAP+" library="wirepad" deviceset="2,54/0,8" device=""/>
-<part name="R47" library="0-rcl" deviceset="R-TRIMM" device="TS63Z"/>
-<part name="R39" library="0-rcl" deviceset="R-TRIMM" device="3314J"/>
 </parts>
 <sheets>
@@
 <wire x1="624.84" y1="68.58" x2="624.84" y2="149.86" width="0.1524" layer="94" style="shortdash"/>
 <text x="640.08" y="71.12" size="2.54" layer="97">RTC Clock</text>
+<text x="177.8" y="53.34" size="1.778" layer="91">todo: add jumper here</text>
 </plain>
 <instances>
@@
 <instance part="CAP-" gate="P" x="678.18" y="142.24" rot="R270"/>
 <instance part="CAP+" gate="P" x="670.56" y="142.24" rot="R270"/>
-<instance part="R47" gate="G$1" x="190.5" y="68.58"/>
-<instance part="R39" gate="G$1" x="190.5" y="83.82"/>
 </instances>
 <busses>

Commit message: updates in part values
Parts:
- IC1: value TL5626D -> TLV5626D
- R16, R24: value 2M2 -> 1M
- R17, R25: value 4M7 -> 1M
- R21, R29: value 500K -> 5K
- R22, R30: value 33K -> 10K
Changed lines of the file:
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@@
 <part name="R12" library="0-rcl" deviceset="R-TRIMM" device="4G/J" value="500K"/>
 <part name="R13" library="rcl" deviceset="R-EU_" device="R0805S" value="2M"/>
-<part name="R16" library="rcl" deviceset="R-EU_" device="R0805S" value="2M2"/>
-<part name="R17" library="rcl" deviceset="R-EU_" device="R0805S" value="4M7"/>
+<part name="R16" library="rcl" deviceset="R-EU_" device="R0805S" value="1M"/>
+<part name="R17" library="rcl" deviceset="R-EU_" device="R0805S" value="1M"/>
 <part name="Q1" library="SparkFun" deviceset="TRANSISTOR_NPN" device="SOT23-3"/>
 <part name="Q3" library="SparkFun" deviceset="TRANSISTOR_NPN" device="SOT23-3"/>
@@
 <part name="C15" library="rcl" deviceset="CPOL-EU" device="SMCB" value="10uF"/>
 <part name="R20" library="0-rcl" deviceset="R-TRIMM" device="4G/J" value="10K"/>
-<part name="R21" library="0-rcl" deviceset="R-TRIMM" device="4G/J" value="500K"/>
-<part name="R22" library="rcl" deviceset="R-EU_" device="R0805S" value="33K"/>
+<part name="R21" library="0-rcl" deviceset="R-TRIMM" device="4G/J" value="5K"/>
+<part name="R22" library="rcl" deviceset="R-EU_" device="R0805S" value="10K"/>
 <part name="R23" library="rcl" deviceset="R-EU_" device="R0805S" value="0"/>
 <part name="GND19" library="supply1" deviceset="GND" device=""/>
@@
 <part name="V3" library="supply2" deviceset="+5V" device=""/>
 <part name="V4" library="supply2" deviceset="+5V" device=""/>
-<part name="R24" library="rcl" deviceset="R-EU_" device="R0805S" value="2M2"/>
-<part name="R25" library="rcl" deviceset="R-EU_" device="R0805S" value="4M7"/>
+<part name="R24" library="rcl" deviceset="R-EU_" device="R0805S" value="1M"/>
+<part name="R25" library="rcl" deviceset="R-EU_" device="R0805S" value="1M"/>
 <part name="Q5" library="SparkFun" deviceset="TRANSISTOR_NPN" device="SOT23-3"/>
 <part name="Q6" library="SparkFun" deviceset="TRANSISTOR_NPN" device="SOT23-3"/>
@@
 <part name="C18" library="rcl" deviceset="CPOL-EU" device="SMCB" value="10uF"/>
 <part name="R28" library="0-rcl" deviceset="R-TRIMM" device="4G/J" value="10K"/>
-<part name="R29" library="0-rcl" deviceset="R-TRIMM" device="4G/J" value="500K"/>
-<part name="R30" library="rcl" deviceset="R-EU_" device="R0805S" value="33K"/>
+<part name="R29" library="0-rcl" deviceset="R-TRIMM" device="4G/J" value="5K"/>
+<part name="R30" library="rcl" deviceset="R-EU_" device="R0805S" value="10K"/>
 <part name="R31" library="rcl" deviceset="R-EU_" device="R0805S" value="0"/>
 <part name="GND24" library="supply1" deviceset="GND" device=""/>
@@
 <part name="V5" library="supply2" deviceset="+5V" device=""/>
 <part name="V9" library="supply2" deviceset="+5V" device=""/>
-<part name="IC1" library="0-tlv5626" deviceset="TL5626*" device="D"/>
+<part name="IC1" library="0-tlv5626" deviceset="TL5626*" device="D" value="TLV5626D"/>
 <part name="C19" library="rcl" deviceset="C-EU" device="C0603K" value="100nF"/>
 <part name="GND27" library="supply1" deviceset="GND" device=""/>

Commit message: latest fixes for 3loshnik schematics
morsekeyer
Parts:
- R33: value 2M2 -> 470K
- R34: value 75-100K -> 10K
Other:
- note added: "Heater: 1 winding through 0.5ohm series"
Changed lines of the file:
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@@
 <part name="GND35" library="supply1" deviceset="GND" device=""/>
 <part name="Q7" library="SparkFun" deviceset="TRANSISTOR_NPN" device="SOT23-3"/>
-<part name="R33" library="rcl" deviceset="R-EU_" device="R0805S" value="2M2"/>
-<part name="R34" library="rcl" deviceset="R-EU_" device="R0805S" value="75-100K"/>
+<part name="R33" library="rcl" deviceset="R-EU_" device="R0805S" value="470K"/>
+<part name="R34" library="rcl" deviceset="R-EU_" device="R0805S" value="10K"/>
 <part name="GND36" library="supply1" deviceset="GND" device=""/>
 <part name="R35" library="rcl" deviceset="R-EU_" device="R0805S" value="1K"/>
@@
 <text x="640.08" y="71.12" size="2.54" layer="97">RTC Clock</text>
 <text x="177.8" y="53.34" size="1.778" layer="91">todo: add jumper here</text>
+<text x="254" y="109.22" size="1.778" layer="91">Heater: 1 winding through 0.5ohm series</text>
 </plain>
 <instances>

Commit message: zloshnik circuit update (cosmetic)
Other:
- note added: "+12VDC"
- note added: "2x multiplier"
- note added: "3LOSHNIK (Zloshnik)"
- note added: "3x multiplier"
- note added: "A vector CRT display"
- note added: "CRT connector"
- note added: "Central processor"
- note added: "Deflection amplifiers"
- note added: "HV ladder"
- note added: "High-voltage unit"
- note added: "Power supply"
- note added: "TL5626D"
- note added: "TRANSFORMER"
- note added: "Viacheslav Slavinsky, 2012"
- note added: "X/Y DAC"
- note added: "Z modulator"
- note added: "based on 3LO1I tube"
- note added: "http://sensi.org/~svo"
- moved on the sheet: +300V, -450V, C1, C10, C11, C12, C13, C14, C16, C17, C19, C2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
