File: projects/morsekeyer/eagle/morsekeyer/keyer.brd (EAGLE design)
At the start: 42.9 x 52.1 mm, 26 parts, among them IC1 G2X[2/3]1---N14, IC3 REG1117, SW1 BUTTON_6X6_THRU, X1 USB-MICROB, X2 1503_09S5

Commit message: incursion first rev
Parts:
- R33: value 100 -> 150
Changed lines of the file:
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@@
 <element name="C25" library="rcl" package="SMC_B" value="10uF" x="18.7325" y="22.86" rot="MR0"/>
 <element name="Q7" library="SparkFun" package="SOT23-3" value="" x="17.4625" y="43.18" rot="MR0"/>
-<element name="R33" library="rcl" package="R0805-SVO" value="100" x="17.4625" y="48.26" rot="MR270"/>
+<element name="R33" library="rcl" package="R0805-SVO" value="150" x="17.4625" y="48.26" rot="MR270"/>
 <element name="R35" library="rcl" package="R0805-SVO" value="1K" x="31.75" y="40.64" rot="MR90"/>
 <element name="C1" library="rcl" package="D/7343-31R" value="220uF" x="10.16" y="47.625" rot="MR180"/>
