File: projects/morsekeyer/eagle/morsekeyer/keyer.sch (EAGLE design)
At the start: 26 parts, among them IC1 G2X[2/3]1---N14, IC3 REG1117, SW1 BUTTON_6X6_THRU, X1 USB-MICROB, X2 1503_09S5

Commit message: incursion first rev
Parts:
- R33: value 100 -> 150
Changed lines of the file:
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@@
 <part name="GND42" library="supply1" deviceset="GND" device=""/>
 <part name="Q7" library="SparkFun" deviceset="TRANSISTOR_NPN" device="SOT23-3"/>
-<part name="R33" library="rcl" deviceset="R-EU_" device="R0805S" value="100"/>
+<part name="R33" library="rcl" deviceset="R-EU_" device="R0805S" value="150"/>
 <part name="GND36" library="supply1" deviceset="GND" device=""/>
 <part name="R35" library="rcl" deviceset="R-EU_" device="R0805S" value="1K"/>
